File: HTmultipurposeboard.kicad_pcb (KiCad board)
At the start: 4 copper layers, 100 x 60 mm, 117 parts, among them IC1 TPS543620RPYR, J1 USB_C_Receptacle_USB2.0, J11 Conn_01x03, J13 Conn_01x02, J14 Conn_01x02, J2 Conn_01x03, J3 Conn_01x03, J4 Conn_01x03, Q4 BSS138, Q5 BSS138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

Commit message: update
Parts:
- removed C16, C19, C24: 10u, Capacitor_SMD:C_0805_2012Metric_Pad1.18x1.45mm_HandSolder
- removed C27, C28, C30, C34: 0.1u, Capacitor_SMD:C_0402_1005Metric_Pad0.74x0.62mm_HandSolder
- removed C29: 2.2u, Capacitor_SMD:C_0402_1005Metric_Pad0.74x0.62mm_HandSolder
- removed C31: 22p, Capacitor_SMD:C_0402_1005Metric_Pad0.74x0.62mm_HandSolder
- removed C32, C33: 22u, Capacitor_SMD:C_1210_3225Metric_Pad1.33x2.70mm_HandSolder
- removed D18, D29: LED, LED_SMD:LED_0603_1608Metric_Pad1.05x0.95mm_HandSolder
- removed D27, D28: D, 0-Myparts:SS2040FL
- removed IC1: TPS543620RPYR, 0-Myparts:TPS543620RPYR
- removed L1: 1.8u, Inductor_SMD:L_Coilcraft_XAL6030-XXX
- removed L2: 0.47u, Inductor_SMD:L_0603_1608Metric_Pad1.05x0.95mm_HandSolder
- removed R22, R26: R, Resistor_SMD:R_0603_1608Metric_Pad0.98x0.95mm_HandSolder
- removed R23: 88.7k, Resistor_SMD:R_0603_1608Metric_Pad0.98x0.95mm_HandSolder
- removed R24: 19.6k, Resistor_SMD:R_0603_1608Metric_Pad0.98x0.95mm_HandSolder
- removed R25: 100k, Inductor_SMD:L_0603_1608Metric_Pad1.05x0.95mm_HandSolder
- removed R29, R40: 10k, Resistor_SMD:R_0402_1005Metric_Pad0.72x0.64mm_HandSolder
- removed R33, R34, R36, R37: R, Resistor_SMD:R_0402_1005Metric_Pad0.72x0.64mm_HandSolder
- removed R35, R5: 10k, Resistor_SMD:R_0603_1608Metric_Pad0.98x0.95mm_HandSolder
- removed R39: 90.9k, Resistor_SMD:R_0402_1005Metric_Pad0.72x0.64mm_HandSolder
- added C14: 10u, Capacitor_SMD:C_0805_2012Metric_Pad1.18x1.45mm_HandSolder, F.Cu at (117.4, 89.2)
- added C4: 10u, Capacitor_SMD:C_0805_2012Metric_Pad1.18x1.45mm_HandSolder, F.Cu at (77.3, 79.7)
- added C9: 10u, Capacitor_SMD:C_0805_2012Metric_Pad1.18x1.45mm_HandSolder, F.Cu at (77.5, 85.0)
- added U6: AZ1084-5.0, Package_TO_SOT_SMD:TO-252-2, F.Cu at (68.8, 80.1)
- added U7: AZ1084-5.0, Package_TO_SOT_SMD:TO-252-2, F.Cu at (68.7, 97.8)
- added U9: AZ1084-5.0, Package_TO_SOT_SMD:TO-252-2, F.Cu at (68.8, 88.3)
- C11, C15: value 10u -> 22u; footprint Capacitor_SMD:C_0805_2012Metric_Pad1.18x1.45mm_HandSolder -> Capacitor_SMD:C_1206_3216Metric_Pad1.33x1.80mm_HandSolder
- C12: value 4.7u -> 22u; footprint Capacitor_SMD:C_0603_1608Metric_Pad1.08x0.95mm_HandSolder -> Capacitor_SMD:C_1206_3216Metric_Pad1.33x1.80mm_HandSolder
- C13: value 10p -> 22u; footprint Capacitor_SMD:C_0603_1608Metric_Pad1.08x0.95mm_HandSolder -> Capacitor_SMD:C_1206_3216Metric_Pad1.33x1.80mm_HandSolder
- C20: moved to B.Cu
- U8: value TPS628511DRLR -> LT1963AxST-3.3; footprint 0_kicadlib:DRL0008A-MFG -> Package_TO_SOT_SMD:SOT-223-3_TabPin2
- moved C11 61.4 mm to (64.7, 72.5), turned to 90 degrees
- moved C13 55.4 mm to (68.7, 103.1), turned to 0 degrees
- moved C10 45.2 mm to (76.7, 95.7)
- moved C12 44.9 mm to (78.3, 91.5)
- moved C15 13.1 mm to (118.0, 99.1), turned to 0 degrees
- moved C20 4.95 mm to (81.3, 88.3), turned to 180 degrees
- moved R31 4.08 mm to (101.9, 74.3)
- moved U8 1.86 mm to (120.0, 94.2), turned to 0 degrees
- moved C7 1.10 mm to (120.5, 77.8), turned to 180 degrees
- moved R27 0.53 mm to (100.3, 74.3)
Connections:
- net +5P renamed Net-(D13-A)
- C10 pad 1: Net-(D27-K) -> +BATT
- C10 pad 2: GNDD -> GNDA
- C11 pad 1: Net-(D27-K) -> +5F
- C11 pad 2: GNDD -> GNDA
- C12 pad 1: Net-(U8-SS_TR) -> +5C
- C12 pad 2: GNDD -> GNDA
- C13 pad 1: +3.3V -> +5VA
- C13 pad 2: Net-(U8-FB) -> GNDA
- C15 pad 2: GNDD -> GNDA
- C22 pad 2: GNDA -> GNDPWR
- C26 pad 2: GNDA -> GNDPWR
- C38 pad 2: GNDA -> GNDPWR
- C39 pad 2: GNDA -> GNDPWR
- C40 pad 2: GNDA -> GNDPWR
- C7 pad 2: GNDA -> GNDPWR
- J11 pad 3: GNDA -> GNDPWR
- J2 pad 3: GNDA -> GNDPWR
- J3 pad 2: +5VA -> +5F
- J3 pad 3: GNDA -> GNDPWR
- J4 pad 2: +5VA -> +5C
- J4 pad 3: GNDA -> GNDPWR
- R27 pad 2: GNDA -> GNDPWR
- R28 pad 2: GNDA -> GNDPWR
- R9 pad 2: GNDA -> GNDPWR
- U10 pad 1: GNDA -> GNDPWR
- U12 pad 15: GNDA -> GNDPWR
- U12 pad 9: GNDA -> GNDPWR
- U13 pad 15: GNDA -> GNDPWR
- U13 pad 9: GNDA -> GNDPWR
- U14 pad 18: GNDA -> GNDPWR
- U14 pad 19: GNDA -> GNDPWR
- U14 pad 20: GNDA -> GNDPWR
- U14 pad 26: GNDA -> GNDPWR
- U14 pad 27: GNDA -> GNDPWR
- U14 pad 28: GNDA -> GNDPWR
- U18 pad 18: GNDA -> GNDPWR
- U18 pad 19: GNDA -> GNDPWR
- U18 pad 20: GNDA -> GNDPWR
- U18 pad 26: GNDA -> GNDPWR
- U18 pad 27: GNDA -> GNDPWR
- U18 pad 28: GNDA -> GNDPWR
- U4 pad 18: GNDA -> GNDPWR
- U4 pad 19: GNDA -> GNDPWR
- U4 pad 20: GNDA -> GNDPWR
- U4 pad 26: GNDA -> GNDPWR
- U4 pad 27: GNDA -> GNDPWR
- U4 pad 28: GNDA -> GNDPWR
- U5 pad 15: GNDA -> GNDPWR
- U5 pad 9: GNDA -> GNDPWR
- U8 pad 1: Net-(D27-K) -> +5V
- U8 pad 2: Net-(D27-K) -> GNDA
- U8 pad 3: Net-(D27-K) -> +3.3V
Routing:
- net +BATT: track 42.7 -> 89.4 mm, vias 218 -> 177
- net pwm_9: track 46.6 -> 0.00 mm, vias 1 -> 0
- net servo1: track 45.4 -> 0.00 mm, vias 1 -> 0
- net pwm_2: track 45.2 -> 0.00 mm, vias 1 -> 0
- net servo2: track 44.4 -> 0.00 mm, vias 1 -> 0
- net servo3: track 41.9 -> 0.00 mm, vias 1 -> 0
- net pwm_1: track 39.1 -> 0.00 mm, vias 1 -> 0
- net pwm_5: track 38.2 -> 0.00 mm, vias 1 -> 0
- net pwm_8: track 37.0 -> 0.00 mm, vias 1 -> 0
- net +5VA: track 81.8 -> 116.4 mm, vias 0 -> 4
- net +5V: track 97.7 -> 63.8 mm, vias 4 -> 3
- net +5C: track 0.00 -> 17.0 mm
- net +5F: track 0.00 -> 12.0 mm
- net Net-(IC1-EN): track 9.34 -> 0.00 mm
- net Net-(IC1-BP5): track 9.09 -> 0.00 mm, vias 2 -> 0
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- added copper zone on B.Cu, net GNDA
- added copper zone on In1.Cu, net GNDA
- removed copper zone on F.Cu, net +5VA
- removed copper zone on F.Cu, net Net-(D27-K)
Other:
- outline, holes or cut-outs redrawn

Commit message: アホみたいにフラストレーションが溜まってるので寝る
Parts:
- added C16: 1u, Capacitor_SMD:C_0603_1608Metric_Pad1.08x0.95mm_HandSolder, F.Cu at (94.0, 86.7)
- added C19: 10u, Capacitor_SMD:C_0805_2012Metric_Pad1.18x1.45mm_HandSolder, F.Cu at (93.4, 83.8)
- added R10: 1K, Resistor_SMD:R_0603_1608Metric_Pad0.98x0.95mm_HandSolder, F.Cu at (125.9, 85.8)
- added R11: 1K, Resistor_SMD:R_0603_1608Metric_Pad0.98x0.95mm_HandSolder, F.Cu at (108.7, 79.9)
- added R12: 1K, Resistor_SMD:R_0603_1608Metric_Pad0.98x0.95mm_HandSolder, F.Cu at (112.2, 79.9)
- added R13: 1K, Resistor_SMD:R_0603_1608Metric_Pad0.98x0.95mm_HandSolder, F.Cu at (112.2, 77.0)
- added R14: 1K, Resistor_SMD:R_0603_1608Metric_Pad0.98x0.95mm_HandSolder, F.Cu at (108.7, 77.0)
- added R15: 1K, Resistor_SMD:R_0603_1608Metric_Pad0.98x0.95mm_HandSolder, F.Cu at (108.6, 85.9)
- added R16: 1K, Resistor_SMD:R_0603_1608Metric_Pad0.98x0.95mm_HandSolder, F.Cu at (112.1, 85.9)
- added R17: 1K, Resistor_SMD:R_0603_1608Metric_Pad0.98x0.95mm_HandSolder, F.Cu at (115.7, 85.9)
- added R19: 1K, Resistor_SMD:R_0603_1608Metric_Pad0.98x0.95mm_HandSolder, F.Cu at (112.2, 82.9)
- added R21: 1K, Resistor_SMD:R_0603_1608Metric_Pad0.98x0.95mm_HandSolder, F.Cu at (108.7, 82.9)
- added R5: 1K, Resistor_SMD:R_0603_1608Metric_Pad0.98x0.95mm_HandSolder, F.Cu at (123.1, 85.7)
- added R7: 1K, Resistor_SMD:R_0603_1608Metric_Pad0.98x0.95mm_HandSolder, F.Cu at (123.1, 89.3)
- added R8: 1K, Resistor_SMD:R_0603_1608Metric_Pad0.98x0.95mm_HandSolder, F.Cu at (125.9, 89.3)
- added U15: ~, Package_SO:SSOP-16_3.9x4.9mm_P0.635mm, F.Cu at (101.2, 84.9)
- U13: value Si8640BB-B-IS1 -> AP7375-33SA-7; footprint Package_SO:SSOP-16_3.9x4.9mm_P0.635mm -> Package_TO_SOT_SMD:SOT-23
- moved U13 8.60 mm to (94.0, 89.6), turned to 90 degrees
- moved C15 6.90 mm to (124.0, 95.7), turned to 90 degrees
- moved C14 6.24 mm to (111.6, 91.5), turned to 180 degrees
- moved C26 2.33 mm to (96.8, 84.9), turned to 90 degrees
- moved U8 1.80 mm to (118.7, 95.5), turned to 90 degrees
Connections:
- C22 pad 1: +5VA -> Vdrive
- C26 pad 1: +5VA -> Vdrive
- C7 pad 1: +5VA -> Vdrive
- U12 pad 10: +5VA -> Vdrive
- U12 pad 16: +5VA -> Vdrive
- U13 pad 1: +3.3V -> +BATT
- U13 pad 2: GNDD -> Vdrive
- U13 pad 3: servo3 -> Net-(U13-GND)
- U18 pad 4: Net-(U13-B4) -> Net-(U15-B5)
- U5 pad 10: +5VA -> Vdrive
- U5 pad 16: +5VA -> Vdrive
Routing:
- net Vdrive: track 0.00 -> 56.8 mm
- net +5VA: track 116.4 -> 62.0 mm, vias 4 -> 2
- net RGB_OUTPUT_VCC: track 0.00 -> 51.3 mm, vias 0 -> 1
- net Net-(U15-B5): track 0.00 -> 40.4 mm, vias 0 -> 2
- net Net-(U13-B4): track 40.4 -> 0.00 mm, vias 2 -> 0
- net servo2: track 0.00 -> 11.7 mm
- net +5V: track 63.8 -> 75.4 mm
- net servo3: track 0.00 -> 8.41 mm
- net pwm_5: track 0.00 -> 8.22 mm
- net servo1: track 0.00 -> 8.22 mm
- net pwm_1: track 0.00 -> 7.94 mm
- net pwm_6: track 0.00 -> 6.45 mm
- net GNDA: track 16.1 -> 9.75 mm
- net pwm_3: track 0.00 -> 6.25 mm
- net +BATT: track 89.4 -> 95.2 mm
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
Commit message: update
Connections:
- R30 pad 1: +5VA -> +5F
- R31 pad 1: +5VA -> +5F
- R32 pad 1: +5VA -> +5F
Routing:
- net +5V: track 75.4 -> 55.9 mm
- net pwm_7: track 2.03 -> 12.3 mm
- net pwm_6: track 6.45 -> 15.7 mm
- net +5F: track 12.0 -> 21.2 mm, vias 0 -> 2
- net Net-(U12-B4): track 0.00 -> 9.22 mm
- net +5VA: track 62.0 -> 58.4 mm, vias 2 -> 0
- net +3.3V: track 150.7 -> 148.9 mm
- net Net-(U14-INB): track 26.2 -> 25.5 mm
