File: HTmultipurposeboard.kicad_sch (KiCad schematic)
At the start: 113 parts, among them IC1 TPS543620RPYR, J1 USB_C_Receptacle_USB2.0, J11 Conn_01x03, J13 Conn_01x02, J14 Conn_01x02, J2 Conn_01x03, J3 Conn_01x03, J4 Conn_01x03, Q4 BSS138, Q5 BSS138, SW1 SW_Push, SW3 SW_Push, U1 xh2pin, U10 MCWI05-12S05, U11 CH340K, U12 Si8640BB-B-IS1, U13 Si8640BB-B-IS1, U14 VNH5019A-E, U18 VNH5019A-E, U2 ESP32-WROOM-32D, U3 xh2pin, U4 VNH5019A-E, U5 Si8640BB-B-IS1, U8 TPS628511DRLR

Commit message: update
Parts:
- removed C16, C19, C24: 10u, Capacitor_SMD:C_0805_2012Metric_Pad1.18x1.45mm_HandSolder, symbol Device:C
- removed C27, C28, C30, C34: 0.1u, Capacitor_SMD:C_0402_1005Metric_Pad0.74x0.62mm_HandSolder, symbol Device:C
- removed C29: 2.2u, Capacitor_SMD:C_0402_1005Metric_Pad0.74x0.62mm_HandSolder, symbol Device:C
- removed C31: 22p, Capacitor_SMD:C_0402_1005Metric_Pad0.74x0.62mm_HandSolder, symbol Device:C
- removed C32, C33: 22u, Capacitor_SMD:C_1210_3225Metric_Pad1.33x2.70mm_HandSolder, symbol Device:C
- removed D18, D29: LED, LED_SMD:LED_0603_1608Metric_Pad1.05x0.95mm_HandSolder, symbol Device:LED
- removed D27, D28: D, 0-Myparts:SS2040FL, symbol Device:D
- removed IC1: TPS543620RPYR, 0-Myparts:TPS543620RPYR, symbol 0_symbols:TPS543620RPYR
- removed L1: 1.8u, Inductor_SMD:L_Coilcraft_XAL6030-XXX, symbol Device:L
- removed L2: 0.47u, Inductor_SMD:L_0603_1608Metric_Pad1.05x0.95mm_HandSolder, symbol Device:L
- removed R22, R26: R, Resistor_SMD:R_0603_1608Metric_Pad0.98x0.95mm_HandSolder, symbol Device:R
- removed R23: 88.7k, Resistor_SMD:R_0603_1608Metric_Pad0.98x0.95mm_HandSolder, symbol Device:R
- removed R24: 19.6k, Resistor_SMD:R_0603_1608Metric_Pad0.98x0.95mm_HandSolder, symbol Device:R
- removed R25: 100k, Inductor_SMD:L_0603_1608Metric_Pad1.05x0.95mm_HandSolder, symbol Device:R
- removed R29, R40: 10k, Resistor_SMD:R_0402_1005Metric_Pad0.72x0.64mm_HandSolder, symbol Device:R
- removed R33, R34, R36, R37: R, Resistor_SMD:R_0402_1005Metric_Pad0.72x0.64mm_HandSolder, symbol Device:R
- removed R35, R5: 10k, Resistor_SMD:R_0603_1608Metric_Pad0.98x0.95mm_HandSolder, symbol Device:R
- removed R39: 90.9k, Resistor_SMD:R_0402_1005Metric_Pad0.72x0.64mm_HandSolder, symbol Device:R
- removed U8: TPS628511DRLR, 0_kicadlib:DRL0008A-MFG, symbol 0_symbols:TPS628511DRLR
- added C14, C4, C9: 10u, Capacitor_SMD:C_0805_2012Metric_Pad1.18x1.45mm_HandSolder, symbol Device:C
- added U6, U7, U9: AZ1084-5.0, Package_TO_SOT_SMD:TO-252-2, symbol Regulator_Linear:AZ1084-5.0
- added U8: LT1963AxST-3.3, Package_TO_SOT_SMD:SOT-223-3_TabPin2, symbol Regulator_Linear:LT1963AxST-3.3
- C11, C15: value 10u -> 22u; footprint Capacitor_SMD:C_0805_2012Metric_Pad1.18x1.45mm_HandSolder -> Capacitor_SMD:C_1206_3216Metric_Pad1.33x1.80mm_HandSolder
- C12: value 4.7u -> 22u; footprint Capacitor_SMD:C_0603_1608Metric_Pad1.08x0.95mm_HandSolder -> Capacitor_SMD:C_1206_3216Metric_Pad1.33x1.80mm_HandSolder
- C13: value 10p -> 22u; footprint Capacitor_SMD:C_0603_1608Metric_Pad1.08x0.95mm_HandSolder -> Capacitor_SMD:C_1206_3216Metric_Pad1.33x1.80mm_HandSolder
Connections:
- net +3.3V: now also U8.3 (OUT); no longer C13.1
- net +5V: now also C14.1, U8.1 (IN)
- net +5VA: now also C13.1, U7.2 (VO); no longer J3.2 (Pin_2), J4.2 (Pin_2)
- net +BATT: now also C10.1, C4.1, C9.1, U6.3 (VI), U7.3 (VI), U9.3 (VI)
- net GNDA: now also C10.2, C11.2, C12.2, C13.2, C15.2, C14.2, C4.2, C9.2, U6.1 (GND), U7.1 (GND), U8.2 (GND), U9.1 (GND); no longer C22.2, C26.2, C38.2, C39.2, C40.2, C7.2, J11.3 (Pin_3), J2.3 (Pin_3), J3.3 (Pin_3), J4.3 (Pin_3), R27.2, R28.2, R9.2, U10.1 (-Vin), U12.15 (GND2), U12.9 (GND2), U13.15 (GND2), U13.9 (GND2), U14.18 (GNDB), U14.19 (GNDB), U14.20 (GNDB), U14.26 (GNDA), U14.27 (GNDA), U14.28 (GNDA), U18.18 (GNDB), U18.19 (GNDB), U18.20 (GNDB), U18.26 (GNDA), U18.27 (GNDA), U18.28 (GNDA), U4.18 (GNDB), U4.19 (GNDB), U4.20 (GNDB), U4.26 (GNDA), U4.27 (GNDA), U4.28 (GNDA), U5.15 (GND2), U5.9 (GND2)
- net GNDD: no longer C10.2, C11.2, C12.2, C15.2
- net +5C: now reaches C12.1
- net +5C: now also J4.2 (Pin_2), U9.2 (VO)
- net +5F: now reaches C11.1
- net +5F: now also J3.2 (Pin_2), U6.2 (VO); no longer C10.1
- net +5P: no longer names the net of C18.1, D13.2 (A), U10.6 (+Vout)
- new net GNDPWR: C22.2, C26.2, C38.2, C39.2, C40.2, C7.2, J11.3 (Pin_3), J2.3 (Pin_3), J3.3 (Pin_3), J4.3 (Pin_3), R27.2, R28.2, R9.2, U10.1 (-Vin), U12.15 (GND2), U12.9 (GND2), U13.15 (GND2), U13.9 (GND2), U14.18 (GNDB), U14.19 (GNDB), U14.20 (GNDB), U14.26 (GNDA), U14.27 (GNDA), U14.28 (GNDA), U18.18 (GNDB), U18.19 (GNDB), U18.20 (GNDB), U18.26 (GNDA), U18.27 (GNDA), U18.28 (GNDA), U4.18 (GNDB), U4.19 (GNDB), U4.20 (GNDB), U4.26 (GNDA), U4.27 (GNDA), U4.28 (GNDA), U5.15 (GND2), U5.9 (GND2)
Other:
- moved on the sheet: C18, C38, C39, C40, D13, D17, J3, J4, U10

Commit message: アホみたいにフラストレーションが溜まってるので寝る
Parts:
- removed U13: Si8640BB-B-IS1, Package_SO:SSOP-16_3.9x4.9mm_P0.635mm, symbol Isolator:Si8640BB-B-IS1
- added C16: 1u, Capacitor_SMD:C_0603_1608Metric_Pad1.08x0.95mm_HandSolder, symbol Device:C
- added C19: 10u, Capacitor_SMD:C_0805_2012Metric_Pad1.18x1.45mm_HandSolder, symbol Device:C
- added R10, R11, R12, R13, R14, R15, R16, R17, R19, R21, R5, R7, R8: 1K, Resistor_SMD:R_0603_1608Metric_Pad0.98x0.95mm_HandSolder, symbol Device:R
- added U13: AP7375-33SA-7, Package_TO_SOT_SMD:SOT-23, symbol 0_symbols:AP7375-33SA-7
- added U15: ~, Package_SO:SSOP-16_3.9x4.9mm_P0.635mm, symbol 0_symbols:SI8650AB-B-IS1
Connections:
- net +3.3V: now also U15.1 (VDD1)
- net +5VA: no longer C22.1, C26.1, C7.1, U12.10 (EN2), U12.16 (VDD2), U5.10 (EN2), U5.16 (VDD2)
- net +BATT: now also C16.1, U13.1 (VIN)
- net GNDD: now also R10.2, R11.2, R12.2, R13.2, R14.2, R15.2, R16.2, R17.2, R19.2, R21.2, R5.2, R7.2, R8.2, U15.8 (GND1)
- net GNDPWR: now also U15.9 (GND2)
- net IO25_WS2812: now also R15.1, U15.2 (A1)
- net RGB_OUTPUT_VCC: now also U15.15 (B1)
- net SERVO_1: now also U15.12 (B4)
- net SERVO_2: now also U15.13 (B3)
- net SERVO_3: now also U15.14 (B2)
- net pwm_1: now also R12.1
- net pwm_2: now also R11.1
- net pwm_3: now also R7.1
- net pwm_4: now also R5.1
- net pwm_5: now also R13.1
- net pwm_6: now also R8.1
- net pwm_7: now also R10.1
- net pwm_8: now also R14.1
- net pwm_9: now also R21.1, U15.6 (A5)
- net servo1: now also R19.1, U15.5 (A4)
- net servo2: now also R17.1, U15.4 (A3)
- net servo3: now also R16.1, U15.3 (A2)
- net at U18.4 (INA): now also U15.11 (B5)
- new net: C16.2, C19.2, U13.3 (GND)
- new net Vdrive: C19.1, C22.1, C26.1, C7.1, U12.10 (EN2), U12.16 (VDD2), U13.2 (VOUT), U15.10 (EN2), U15.16 (VDD2), U5.10 (EN2), U5.16 (VDD2)

Commit message: update
Connections:
- net +5F: now also R30.1, R31.1, R32.1
- net +5VA: no longer R30.1, R31.1, R32.1
